File: base/base.kicad_pcb (KiCad board)
At the start: 2 copper layers, 21.5 x 13 mm, 3 parts, among them J1 Conn_Coaxial, J2 Conn_Coaxial

Commit message: Update based on first constructed version
Routing:
- net GND: track 1.08 -> 0.07 mm
Changed lines of the file:
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@@
 	)
 	(segment
-		(start 139 81.3125)
-		(end 138.999999 80.230445)
+		(start 139 79.65)
+		(end 138.95 79.6)
 		(width 0.2)
 		(layer "F.Cu")
@@
 	)
 	(via
-		(at 139 86.5)
+		(at 138.95 86.75)
 		(size 0.6)
 		(drill 0.3)
@@
 	)
 	(via
-		(at 138.999999 80.230445)
+		(at 138.95 79.6)
 		(size 0.6)
 		(drill 0.3)
@@
 	)
 	(via
-		(at 139 82.5)
+		(at 139 83.05)
 		(size 0.6)
 		(drill 0.3)
