File: base/base.kicad_sch (KiCad schematic)
At the start: 3 parts, among them J1 Conn_Coaxial, J2 Conn_Coaxial

Commit message: Update based on first constructed version
Changed lines of the file:
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@@
 				)
 				(justify left)
+				(hide yes)
 			)
 		)
@@
 				)
 				(justify left)
+				(hide yes)
 			)
 		)
